File: pcb/mainboard.kicad_sch (KiCad schematic)
At the start: 12 parts

Commit message: updating schematic diagram
Parts:
- removed J?: ESP32 WROOM 32U, symbol Connector:Conn_01x19_Female
- removed J?: DevKit C V4, symbol Connector:Conn_01x19_Female
- added U?: ESP32-DevKitC, Espressif:ESP32-DevKitC, symbol Espressif:ESP32-DevKitC
Connections:
- net IN3 is gone; now on an unnamed net: J?.1 (Pin_1)
- net at J?.3 (Pin_3): now also J?.2 (Pin_2), R?.1, R?.2, R?.2, R?.2, U?.38 (GND)
- net at J?.4 (Pin_4): now also J?.1 (Pin_1), J?.1 (Pin_1), U?.1 (3V3)
- removed net GND: J?.2 (Pin_2), J?.2 (Pin_2), R?.1, R?.2, R?.2, R?.2
- net IN1: no longer names the net of J?.2 (Pin_2), R?.1
- net IN1: now also U?.10 (DAC_2/ADC2_CH9/GPIO26)
- net IN2: no longer names the net of J?.2 (Pin_2), R?.1
- net IN2: now also U?.11 (ADC2_CH7/GPIO27)
- removed net OUT1: J?.1 (Pin_1), J?.1 (Pin_1), J?.1 (Pin_1), J?.3 (Pin_3)
- net OUT2: no longer names the net of D?.2 (A)
- net OUT2: now also U?.9 (DAC_1/ADC2_CH8/GPIO25)
- net OUT3: no longer names the net of D?.2 (A)
- net OUT3: now also U?.30 (GPIO18)
- new net: J?.1 (Pin_1), U?.33 (GPIO21)
- new net: J?.2 (Pin_2), U?.36 (GPIO22)
- new net: J?.3 (Pin_3), U?.28 (GPIO17)
Other:
- moved on the sheet: D?, J?, R?
